Commit message: Added SLAM Toolkit config

File: install/bot/share/bot/urdf/robot.xacro (robot description, xacro)
@@ -446,4 +446,10 @@
 </link>
 <link name="camera_link_optical"></link>
+<link name="base_footprint"></link>
+<joint name="base_footprint_joint" type="fixed">
+  <parent link="base_link"/>
+  <child link="base_footprint"/>
+  <origin xyz="0 0 0" rpy="0 0 0"/>
+</joint>
 <joint name="camera_optical_joint" type="fixed">
   <parent link="realsense_link"/>

Commit message: Fixed wheel and castor bugs

File: install/bot/share/bot/urdf/robot.xacro (robot description, xacro)
@@ -467,5 +467,5 @@
   <parent link="base_link"/>
   <child link="right_wheel_link_1"/>
-  <axis xyz="0.00034 -1.0 -0.0"/>
+  <axis xyz="0.00034 1.0 -0.0"/>
 </joint>
 <joint name="camera_mount_joint" type="revolute">
