Commit message: Added PointClound2 and Depth Image

File: install/bot/share/bot/urdf/depth_camera.xacro (robot description, xacro)
@@ -1,5 +1,5 @@
 <?xml version="1.0"?>
 <robot xmlns:xacro="http://www.ros.org/wiki/xacro" >
-    <gazebo reference="vision_module_link_1">
+    <gazebo reference="realsense_link">
         <material>Gazebo/Red</material>
         <sensor name="camera" type="depth">
@@ -10,5 +10,5 @@
                 <horizontal_fov>1.089</horizontal_fov>
                 <image>
-                    <format>R8G8B8</format>
+                    <format>B8G8R8</format>
                     <width>640</width>
                     <height>480</height>
@@ -19,6 +19,6 @@
                 </clip>
             </camera>
-            <plugin name="camera_controller" filename="libgazebo_ros_camera.so">
-                <frame_name>realsense_DCAM_1</frame_name>
+            <plugin name="camera_cotroller" filename="libgazebo_ros_camera.so">
+                <frame_name>camera_link_optical</frame_name>
                 <min_depth>0.1</min_depth>
                 <max_depth>100.0</max_depth>

File: src/bot/urdf/depth_camera.xacro (robot description, xacro)
@@ -1,5 +1,5 @@
 <?xml version="1.0"?>
 <robot xmlns:xacro="http://www.ros.org/wiki/xacro" >
-    <gazebo reference="realsense_DCAM_1">
+    <gazebo reference="realsense_link">
         <material>Gazebo/Red</material>
         <sensor name="camera" type="depth">
@@ -10,5 +10,5 @@
                 <horizontal_fov>1.089</horizontal_fov>
                 <image>
-                    <format>R8G8B8</format>
+                    <format>B8G8R8</format>
                     <width>640</width>
                     <height>480</height>
@@ -19,6 +19,6 @@
                 </clip>
             </camera>
-            <plugin name="camera_controller" filename="libgazebo_ros_camera.so">
-                <frame_name>realsense_DCAM_1</frame_name>
+            <plugin name="camera_cotroller" filename="libgazebo_ros_camera.so">
+                <frame_name>camera_link_optical</frame_name>
                 <min_depth>0.1</min_depth>
                 <max_depth>100.0</max_depth>

File: src/bot/urdf/out.urdf (robot description, URDF)
Before this commit: robot robot, 22 links, 21 joints
Links:
- removed link realsense_DCAM_1
- added link realsense_link, mass 0.03866336197375993; collision mesh filename=file:///home/arvi/bot_ws/install/robot_description/share/ro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 scale=0.001 0.001 0.001; visual mesh filename=file:///home/arvi/bot_ws/install/robot_description/share/ro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 scale=0.001 0.001 0.001
Joints:
- joint realsense_joint: child realsense_DCAM_1 -> realsense_link

File: src/bot/urdf/robot.urdf (robot description, URDF)
Before this commit: robot robot, 22 links, 21 joints
Links:
- removed link realsense_DCAM_1
- added link realsense_link, mass 0.03866336197375993; collision mesh filename=file:///home/arvi/ws/install/bot/share/bot/meshes/realsense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 scale=0.001 0.001 0.001; visual mesh filename=file:///home/arvi/ws/install/bot/share/bot/meshes/realsense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 scale=0.001 0.001 0.001
Joints:
- joint realsense_joint: child realsense_DCAM_1 -> realsense_link

File: src/bot/urdf/robot.xacro (robot description, xacro)
@@ -105,5 +105,5 @@
   </collision>
 </link>
-<link name="realsense_DCAM_1">
+<link name="realsense_link">
   <inertial>
     <origin xyz="0.011657410142899255 -0.0011559566930996867 0.0010283014584634431" rpy="0 0 0"/>
@@ -114,5 +114,5 @@
     <origin xyz="-0.073593 0.005001 -0.950168" rpy="0 0 0"/>
     <geometry>
-      <mesh filename="file://$(find robot_description)/meshes/realsense_DCAM_1.stl" scale="0.001 0.001 0.001"/>
+      <mesh filename="file://$(find robot_description)/meshes/realsense_link.stl" scale="0.001 0.001 0.001"/>
     </geometry>
     <material name="silver"/>
@@ -121,5 +121,5 @@
     <origin xyz="-0.073593 0.005001 -0.950168" rpy="0 0 0"/>
     <geometry>
-      <mesh filename="file://$(find robot_description)/meshes/realsense_DCAM_1.stl" scale="0.001 0.001 0.001"/>
+      <mesh filename="file://$(find robot_description)/meshes/realsense_link.stl" scale="0.001 0.001 0.001"/>
     </geometry>
   </collision>
@@ -445,4 +445,10 @@
   </collision>
 </link>
+<link name="camera_link_optical"></link>
+<joint name="camera_optical_joint" type="fixed">
+  <parent link="realsense_link"/>
+  <child link="camera_link_optical"/>
+  <origin xyz="0 0 0" rpy="0 0 -1.5708"/>
+</joint>
 <joint name="left_wheel_joint" type="continuous">
   <origin xyz="-0.0074 0.134581 0.062625" rpy="0 0 0"/>
@@ -472,7 +478,7 @@
 </joint>
 <joint name="realsense_joint" type="fixed">
-  <origin xyz="0.025437 -0.024846 0.048271" rpy="0 0 0"/>
+  <origin xyz="0.025437 -0.024846 0.048271" rpy="${-pi/2} ${-pi/2} ${-pi/2}"/>
   <parent link="vision_module_link_1"/>
-  <child link="realsense_DCAM_1"/>
+  <child link="realsense_link"/>
 </joint>
 <joint name="shoulder_joint" type="continuous">

File: src/robot_description/urdf/robot.xacro (robot description, xacro)
@@ -104,5 +104,5 @@
   </collision>
 </link>
-<link name="realsense_DCAM_1">
+<link name="realsense_link">
   <inertial>
     <origin xyz="0.011657410142899255 -0.0011559566930996867 0.0010283014584634431" rpy="0 0 0"/>
@@ -113,5 +113,5 @@
     <origin xyz="-0.073593 0.005001 -0.950168" rpy="0 0 0"/>
     <geometry>
-      <mesh filename="file://$(find robot_description)/meshes/realsense_DCAM_1.stl" scale="0.001 0.001 0.001"/>
+      <mesh filename="file://$(find robot_description)/meshes/realsense_link.stl" scale="0.001 0.001 0.001"/>
     </geometry>
     <material name="silver"/>
@@ -120,5 +120,5 @@
     <origin xyz="-0.073593 0.005001 -0.950168" rpy="0 0 0"/>
     <geometry>
-      <mesh filename="file://$(find robot_description)/meshes/realsense_DCAM_1.stl" scale="0.001 0.001 0.001"/>
+      <mesh filename="file://$(find robot_description)/meshes/realsense_link.stl" scale="0.001 0.001 0.001"/>
     </geometry>
   </collision>
@@ -473,5 +473,5 @@
   <origin xyz="0.025437 -0.024846 0.048271" rpy="0 0 0"/>
   <parent link="vision_module_link_1"/>
-  <child link="realsense_DCAM_1"/>
+  <child link="realsense_link"/>
 </joint>
 <joint name="shoulder_joint" type="continuous">

Commit message: Map orientation Bug fixes

File: install/bot/share/bot/urdf/depth_camera.xacro (robot description, xacro)
@@ -6,5 +6,5 @@
             <pose> 0 0 0 0 0 0 </pose>
             <visualize>true</visualize>
-            <update_rate>10</update_rate>
+            <update_rate>100</update_rate>
             <camera>
                 <horizontal_fov>1.089</horizontal_fov>
@@ -22,5 +22,5 @@
                 <frame_name>camera_depth_link</frame_name>
                 <min_depth>0.1</min_depth>
-                <max_depth>100.0</max_depth>
+                <max_depth>100</max_depth>
             </plugin>
         </sensor>

File: install/bot/share/bot/urdf/robot.xacro (robot description, xacro)
@@ -461,5 +461,5 @@
   <parent link="camera_depth_link"/>
   <child link="camera_depth_optical_link"/>
-  <origin xyz="0 0 0" rpy="0 0 ${-pi/2} "/>
+  <origin xyz="0 0 0" rpy="${-pi/2} 0 ${-pi/2} "/>
 </joint>
 <joint name="left_wheel_joint" type="continuous">
