Commit message: MInor bug fixes

File: src/bot/urdf/robot.xacro (robot description, xacro)
@@ -455,5 +455,5 @@
   <parent link="realsense_link"/>
   <child link="camera_link_optical"/>
-  <origin xyz="0 0 0" rpy="0 0 -1.5708"/>
+  <origin xyz="0 0 0" rpy="0 -1.5708 0"/>
 </joint>
 <joint name="left_wheel_joint" type="continuous">
@@ -484,5 +484,5 @@
 </joint>
 <joint name="realsense_joint" type="fixed">
-  <origin xyz="0.025437 -0.024846 0.048271" rpy="${-pi/2} ${-pi/2} ${-pi/2}"/>
+  <origin xyz="0.025437 -0.024846 0.048271" rpy="0 0 0"/>
   <parent link="vision_module_link_1"/>
   <child link="realsense_link"/>
